File: kicad_6_docs/CV_generators.kicad_sch (KiCad schematic)
At the start: 22 parts, among them J5 EXPRESSION_PEDAL, U11 TL072, U12 TL072

Commit message: Fix power supply errors, tidy up schematic
Changed lines of the file:
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@@
   (title_block
     (title "Mu-Tron Bi-Phase near-clone")
-    (date "2022-01-14")
+    (date "2022-08-01")
     (rev "0")
     (comment 2 "creativecommons.org/licenses/by/4.0/")
@@
       (effects (font (size 1.27 1.27)) hide)
     )
+    (pin "1")
+    (pin "2")
+    (pin "3")
     (pin "5")
     (pin "6")
     (pin "7")
+    (pin "4")
+    (pin "8")
   )
   (symbol (lib_id "power:+15V") (at 49.53 91.44 0) (unit 1)
@@
     (pin "2")
     (pin "3")
+    (pin "5")
+    (pin "6")
+    (pin "7")
+    (pin "4")
+    (pin "8")
   )
   (symbol (lib_id "Switch:SW_SPDT") (at 77.47 33.02 0) (mirror y) (unit 1)
@@
     (pin "2")
     (pin "3")
+    (pin "5")
+    (pin "6")
+    (pin "7")
+    (pin "4")
+    (pin "8")
   )
   (symbol (lib_id "Device:R_Potentiometer") (at 49.53 30.48 0) (mirror x) (unit 1)
@@
       (effects (font (size 1.27 1.27)) hide)
     )
+    (pin "1")
+    (pin "2")
+    (pin "3")
     (pin "5")
     (pin "6")
     (pin "7")
+    (pin "4")
+    (pin "8")
   )
   (symbol (lib_id "Switch:SW_SPDT") (at 157.48 35.56 0) (mirror y) (unit 1)
@@
     (fill (color 0 0 0 0.0000))
     (property "Sheet name" "LED_driver_B" (id 0) (at 213.36 90.7284 0)
-      (effects (font (size 1.27 1.27)) (justify left bottom))
+      (effects (font (size 1.7 1.7)) (justify left bottom))
     )
     (property "Sheet file" "LED_driver.kicad_sch" (id 1) (at 213.36 130.1246 0)
-      (effects (font (size 1.27 1.27)) (justify left top))
+      (effects (font (size 1.27 1.27)) (justify left top) hide)
     )
     (pin "RAW_CV_IN" input (at 213.36 95.25 180)
@@
     (fill (color 0 0 0 0.0000))
     (property "Sheet name" "LED_driver_A" (id 0) (at 214.63 31.0384 0)
-      (effects (font (size 1.27 1.27)) (justify left bottom))
+      (effects (font (size 1.7 1.7)) (justify left bottom))
     )
     (property "Sheet file" "LED_driver.kicad_sch" (id 1) (at 214.63 70.4346 0)
-      (effects (font (size 1.27 1.27)) (justify left top))
+      (effects (font (size 1.27 1.27)) (justify left top) hide)
     )
     (pin "RAW_CV_IN" input (at 214.63 35.56 180)
@@
     (fill (color 0 0 0 0.0000))
     (property "Sheet name" "LFO_B" (id 0) (at 87.63 93.2684 0)
-      (effects (font (size 1.27 1.27)) (justify left bottom))
+      (effects (font (size 1.7 1.7)) (justify left bottom))
     )
     (property "Sheet file" "LFO.kicad_sch" (id 1) (at 87.63 132.6646 0)
-      (effects (font (size 1.27 1.27)) (justify left top))
+      (effects (font (size 1.27 1.27)) (justify left top) hide)
     )
     (pin "LFO_OUT" output (at 113.03 97.79 0)
@@
     (fill (color 0 0 0 0.0000))
     (property "Sheet name" "LFO_A" (id 0) (at 88.9 28.4984 0)
-      (effects (font (size 1.27 1.27)) (justify left bottom))
+      (effects (font (size 1.7 1.7)) (justify left bottom))
     )
     (property "Sheet file" "LFO.kicad_sch" (id 1) (at 88.9 67.8946 0)
-      (effects (font (size 1.27 1.27)) (justify left top))
+      (effects (font (size 1.27 1.27)) (justify left top) hide)
     )
     (pin "LFO_OUT" output (at 114.3 33.02 0)
