File: kicad_6_docs/phasor.kicad_sch (KiCad schematic)
At the start: 65 parts, among them U10 RC4558, U6 RC4558, U7 RC4558, U8 RC4558, U9 RC4558

Commit message: Fix power supply errors, tidy up schematic
Parts:
- renumbered C17 to C1, C26 to C10, C27 to C11, C28 to C12, C29 to C13, C30 to C14, C31 to C15, C32 to C16, C18 to C2, C19 to C3, C20 to C4, C21 to C5, C22 to C6, C23 to C7, C24 to C8, C25 to C9, R38 to R1, R47 to R10, R48 to R11, R49 to R12, R50 to R13, R51 to R14, R52 to R15, R53 to R16, R54 to R17, R55 to R18, R56 to R19, R39 to R2, R57 to R20, R58 to R21, R59 to R22, R60 to R23, R61 to R24, R62 to R25, R63 to R26, R64 to R27, R65 to R28, R66 to R29, R40 to R3, R67 to R30, R68 to R31, R69 to R32, R70 to R33, R71 to R34, R72 to R35, R73 to R36, R74 to R37, R41 to R4, R42 to R5, R43 to R6, R44 to R7, R45 to R8, R46 to R9, RV3 to RV1, RV4 to RV2, U6 to U1, U7 to U2, U8 to U3, U9 to U4, U10 to U5
Connections:
- net at R1.2, R5.1: now also U1.6 (-); no longer U1.2 (-)
- net at C4.1, R5.2, R7.1: now also U1.7; no longer U1.1
- net at C12.2, R28.2, R29.1: now also U4.5 (+); no longer U4.3 (+)
- net at C1.2, R2.2, R3.1: now also U1.5 (+); no longer U1.3 (+)
- net at C15.1, R32.2, RV2.2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: now also U5.5 (+); no longer U5.3 (+)
- net at C7.2, R16.2, R18.1: now also U3.5 (+); no longer U3.3 (+)
- net at R15.2, R19.1: now also U3.6 (-); no longer U3.2 (-)
- net at C8.1, R14.2, R17.1: now also U2.6 (-); no longer U2.2 (-)
- net at C8.2, C9.1, R17.2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: now also U2.7; no longer U2.1
- net at C14.1, R31.2, R33.1: now also U4.7; no longer U4.1
- net at R27.2, R31.1: now also U4.6 (-); no longer U4.2 (-)
- net at C10.1, R19.2: now also U3.7; no longer U3.1
- net at C6.1, R11.1, R13.1: now also U2.5 (+); no longer U2.3 (+)
- new net: R37.1, U5.6 (-), U5.7
